File: pcb/soundpad.kicad_pcb (KiCad board)
At the start: 2 copper layers, 89.5 x 53 mm, 6 parts, among them SW1 play/pause, SW2 skip, SW3 prev, SW4 volume/mode, U1 MOUDLE-SEEEDUINO-XIAO, U2 ER_OLEDM0.91_1x-I2C

Commit message: PCB fixes
Parts:
- added REF**: MountingHole_3.2mm_M3, MountingHole:MountingHole_3.2mm_M3, F.Cu at (192.5, 77.0)
- added REF**: MountingHole_3.2mm_M3, MountingHole:MountingHole_3.2mm_M3, F.Cu at (122.0, 95.0)
